Commit message: Made a few corrections

File: description/camera.xacro (robot description, xacro)
@@ -16,5 +16,5 @@
    <!--Converting from the ros coordinate system to camera coordinate system
         we rotate the the camera link-->
-    <joint name="camera_joint" type="fixed">
+    <joint name="camera_joint_optical" type="fixed">
         <parent link="camera_link"/>
         <child link="camera_link_optical"/>

File: description/lidar.xacro (robot description, xacro)
@@ -26,5 +26,5 @@
         <sensor name = "laser" type="ray">
             <pose> 0 0 0 0 0 0</pose>
-            <visualize>true</visualize>
+            <visualize>false</visualize>
             <update_rate>10</update_rate>
             <ray>
