Commit message: Made a correction with material

File: description/robot_core.xacro (robot description, xacro)
@@ -3,14 +3,14 @@
     <material name = "white">
         <color rgba = "1 1 1 1"/>
-    </materal>
+    </material>
     <material name = "orange">
         <color rgba = "1 0.3 0.1 1"/>
-    </materal>
+    </material>
     <material name = "blue">
         <color rgba = "0.2 0.2 1 1"/>
-    </materal>
+    </material>
     <material name = "black">
         <color rgba = "0 0 0 1"/>
-    </materal>
+    </material>
     <link name="base_link">
     </link>

Commit message: Correcting error

File: description/robot_core.xacro (robot description, xacro)
@@ -26,4 +26,6 @@
                 <box size= "0.3 0.3 0.15">
             </geometry>
+            <material name = "white">
         </visual>
+    </link>
 </robot>

Commit message: Correcting error with origin of chassis

File: description/robot_core.xacro (robot description, xacro)
@@ -22,9 +22,9 @@
     <link name = "chassis">
         <visual>
-            <origin xyz = "0.15 0.15 0.075"/>
+            <origin xyz = "0.15 0 0.075"/>
             <geometry>
-                <box size= "0.3 0.3 0.15">
+                <box size= "0.3 0.3 0.15"/>
             </geometry>
-            <material name = "white">
+            <material name = "white"/>
         </visual>
     </link>

Commit message: Adding the wheels

File: description/robot_core.xacro (robot description, xacro)
@@ -13,4 +13,5 @@
         <color rgba = "0 0 0 1"/>
     </material>
+    <!-- BASE LINK-->
     <link name="base_link">
     </link>
@@ -18,6 +19,7 @@
         <parent link = "base_link"/>
         <child link = "chassis"/>
-        <origin xyz = "-0.1 0 0"/>
+        <origin xyz = "0.1 0 0"/>
     </joint>
+    <!-- CHASSIS LINK -->
     <link name = "chassis">
         <visual>
@@ -29,3 +31,33 @@
         </visual>
     </link>
+    <!-- LEFT WHEEL LINK-->
+    <joint name = "left_wheel_joint" type ="continuous">
+        <parent link = "base_link"/>
+        <child link = "left_wheel"/>
+        <origin = "0 0.175 0" rpy="-$(pi/2) 0 0"/>
+        <axis = "0 0 1"/>
+    </joint>
+    <link name="left_wheel">
+        <visual>
+            <geometry>
+                <cylinder radius = "0.05" length="0.04">
+            </geometry>
+            <material name = "blue"/>
+        </visual>
+    </link>
+    <!-- RIGHT WHEEL LINK-->
+    <joint name = "right_wheel_joint" type ="continuous">
+        <parent link = "base_link"/>
+        <child link = "right_wheel"/>
+        <origin = "0 -0.175 0" rpy="$(pi/2) 0 0"/>
+        <axis = "0 0 1"/>
+    </joint>
+    <link name="right_wheel">
+        <visual>
+            <geometry>
+                <cylinder radius = "0.05" length="0.04">
+            </geometry>
+            <material name = "blue"/>
+        </visual>
+    </link>
 </robot>

Commit message: Correcting error at left wheel and right wheel

File: description/robot_core.xacro (robot description, xacro)
@@ -35,5 +35,5 @@
         <parent link = "base_link"/>
         <child link = "left_wheel"/>
-        <origin = "0 0.175 0" rpy="-$(pi/2) 0 0"/>
+        <origin xyz= "0 0.175 0" rpy="-$(pi/2) 0 0"/>
         <axis = "0 0 1"/>
     </joint>
@@ -50,5 +50,5 @@
         <parent link = "base_link"/>
         <child link = "right_wheel"/>
-        <origin = "0 -0.175 0" rpy="$(pi/2) 0 0"/>
+        <origin xyz= "0 -0.175 0" rpy="$(pi/2) 0 0"/>
         <axis = "0 0 1"/>
     </joint>

Commit message: Adding the / sign at cylinder

File: description/robot_core.xacro (robot description, xacro)
@@ -36,10 +36,10 @@
         <child link = "left_wheel"/>
         <origin xyz= "0 0.175 0" rpy="-$(pi/2) 0 0"/>
-        <axis = "0 0 1"/>
+        <axis xyz= "0 0 1"/>
     </joint>
     <link name="left_wheel">
         <visual>
             <geometry>
-                <cylinder radius = "0.05" length="0.04">
+                <cylinder radius = "0.05" length="0.04"/>
             </geometry>
             <material name = "blue"/>
@@ -51,10 +51,10 @@
         <child link = "right_wheel"/>
         <origin xyz= "0 -0.175 0" rpy="$(pi/2) 0 0"/>
-        <axis = "0 0 1"/>
+        <axis xyz= "0 0 1"/>
     </joint>
     <link name="right_wheel">
         <visual>
             <geometry>
-                <cylinder radius = "0.05" length="0.04">
+                <cylinder radius = "0.05" length="0.04"/>
             </geometry>
             <material name = "blue"/>

Commit message: Solved the pi problem

File: description/robot_core.xacro (robot description, xacro)
@@ -35,5 +35,5 @@
         <parent link = "base_link"/>
         <child link = "left_wheel"/>
-        <origin xyz= "0 0.175 0" rpy="-$(pi/2) 0 0"/>
+        <origin xyz= "0 0.175 0" rpy="-1.571 0 0"/>
         <axis xyz= "0 0 1"/>
     </joint>
@@ -50,5 +50,5 @@
         <parent link = "base_link"/>
         <child link = "right_wheel"/>
-        <origin xyz= "0 -0.175 0" rpy="$(pi/2) 0 0"/>
+        <origin xyz= "0 -0.175 0" rpy="1.571 0 0"/>
         <axis xyz= "0 0 1"/>
     </joint>

Commit message: Fixed an error

File: description/robot_core.xacro (robot description, xacro)
@@ -19,5 +19,5 @@
         <parent link = "base_link"/>
         <child link = "chassis"/>
-        <origin xyz = "0.1 0 0"/>
+        <origin xyz = "-0.1 0 0"/>
     </joint>
     <!-- CHASSIS LINK -->
@@ -30,4 +30,10 @@
             <material name = "white"/>
         </visual>
+        <collision>
+            <origin xyz = "0.15 0 0.075"/>
+            <geometry>
+                <box size= "0.3 0.3 0.15"/>
+            </geometry>
+        </collision>
     </link>
     <!-- LEFT WHEEL LINK-->
@@ -45,4 +51,9 @@
             <material name = "blue"/>
         </visual>
+        <collision>
+            <geometry>
+                <cylinder radius = "0.05" length="0.04"/>
+            </geometry>
+        </collision>
     </link>
     <!-- RIGHT WHEEL LINK-->
@@ -51,5 +62,5 @@
         <child link = "right_wheel"/>
         <origin xyz= "0 -0.175 0" rpy="1.571 0 0"/>
-        <axis xyz= "0 0 1"/>
+        <axis xyz= "0 0 -1"/>
     </joint>
     <link name="right_wheel">
@@ -60,4 +71,28 @@
             <material name = "blue"/>
         </visual>
+        <collision>
+            <geometry>
+                <cylinder radius = "0.05" length="0.04"/>
+            </geometry>
+        </collision>
+    </link>
+    <!-- CASTER WHEEL LINK-->
+    <joint name = "caster_wheel_joint" type="fixed">
+        <parent link = "chassis"/>
+        <child link = "caster_wheel"/>
+        <origin xyz="0.24 0 0"/>
+    </joint>
+    <link name = "caster_wheel">
+        <visual>
+            <geometry>
+                <sphere radius = "0.05"/>
+            </geometry>
+        <material name = "black"/>
+        </visual>
+        <collision>
+            <geometry>
+                <sphere radius = "0.05"/>
+            </geometry>
+        </collision>
     </link>
 </robot>

Commit message: Done for today

File: description/robot_core.xacro (robot description, xacro)
@@ -1,4 +1,5 @@
 <?xml version="1.0"?>
 <robot xmlns:xacro="http://www.ros.org/wiki/xacro" >
+    <xacro:include filename = "inertial_macros.xacro"/>
     <material name = "white">
         <color rgba = "1 1 1 1"/>
@@ -36,4 +37,7 @@
             </geometry>
         </collision>
+        <xacro:inertial_box mass = "0.5" x="0.3" y="0.3" z="0.15">
+            <origin xyz = "0.15 0 0.075"/>
+        </xacro:inertial_box>
     </link>
     <!-- LEFT WHEEL LINK-->
@@ -56,4 +60,7 @@
             </geometry>
         </collision>
+        <xacro:inertial_cylinder mass="0.1" length="0.04" radius = "0.05">
+            <origin xyz = "0 0 0" rpy = "0 0 0"/>
+        </xacro:inertial_cylinder>
     </link>
     <!-- RIGHT WHEEL LINK-->
@@ -76,4 +83,7 @@
             </geometry>
         </collision>
+        <xacro:inertial_cylinder mass="0.1" length="0.04" radius = "0.05">
+            <origin xyz = "0 0 0" rpy = "0 0 0"/>
+        </xacro:inertial_cylinder>
     </link>
     <!-- CASTER WHEEL LINK-->
@@ -95,4 +105,7 @@
             </geometry>
         </collision>
+        <xacro:inertial_sphere mass="0.1" radius="0.05">
+            <origin xyz = "0 0 0" rpy = "0 0 0"/>
+        </xacro:inertial_sphere>
     </link>
 </robot>

Commit message: Changed the mapper_params file to load my map and to localize

File: description/robot_core.xacro (robot description, xacro)
@@ -16,4 +16,11 @@
     <!-- BASE LINK-->
     <link name="base_link">
+    </link>
+    <joint name="base_footprint_joint" type="fixed">
+        <parent link="base_link"/>
+        <child link="base_footprint"/>
+        <origin xyz="0.0 0.0 0.0" rpy="0.0 0.0 0.0"/>
+    </joint>
+    <link name="base_footprint">
     </link>
     <joint name="chassis_joint" type="fixed">
